File: pd-buddy-wye.sch (KiCad schematic (older format))
At the start: 7 parts, among them J1 Power, J2 UFP, P1 DFP+Power

Commit message: Changed USB-C footprints to CircularHoles variant
Since I plan on getting these made at OSH Park, I shouldn't use
footprints with plated slots.  Now I'm using the CircularHoles
variant of the USB Type-C connector footprint, which is more
OSH-Park-friendly.

This may mean that I need to make a minor board revision after the
footprints are merged.  Not that I mind terribly.
Parts:
- J1, J2: footprint Ratfink_Connectors_USB:USB_C_Receptacle_Amphenol_12401548E4-2A -> Ratfink_Connectors_USB:USB_C_Receptacle_Amphenol_12401548E4-2A_CircularHoles
Changed lines of the file:
@@
 F 0 "J1" H 1100 3650 50  0000 L CNN
 F 1 "Power" H 1900 3650 50  0000 R CNN
-F 2 "Ratfink_Connectors_USB:USB_C_Receptacle_Amphenol_12401548E4-2A" H 1650 2200 50  0001 C CNN
+F 2 "Ratfink_Connectors_USB:USB_C_Receptacle_Amphenol_12401548E4-2A_CircularHoles" H 1650 2200 50  0001 C CNN
 F 3 "" H 1650 2200 50  0001 C CNN
 	1    1500 2200
@@
 F 0 "J2" H 1100 7150 50  0000 L CNN
 F 1 "UFP" H 1900 7150 50  0000 R CNN
-F 2 "Ratfink_Connectors_USB:USB_C_Receptacle_Amphenol_12401548E4-2A" H 1650 5700 50  0001 C CNN
+F 2 "Ratfink_Connectors_USB:USB_C_Receptacle_Amphenol_12401548E4-2A_CircularHoles" H 1650 5700 50  0001 C CNN
 F 3 "" H 1650 5700 50  0001 C CNN
 	1    1500 5700

Commit message: Use connectors from KiCad library
The new USB connector footprints have been merged into the KiCad library
now, so I can use them from there instead of from my own fork.

This bumps the version number to v1.1.  This version is not complete
yet; I plan to make the board a bit smaller before I call the next
version "done".
Parts:
- J1, J2: footprint Ratfink_Connectors_USB:USB_C_Receptacle_Amphenol_12401548E4-2A_CircularHoles -> Connectors_USB:USB_C_Receptacle_Amphenol_12401548E4-2A_CircularHoles
Changed lines of the file:
@@
 Title "PD Buddy Wye"
 Date "2017-08-06"
-Rev "v1.0"
+Rev "v1.1"
 Comp ""
 Comment1 ""
@@
 F 0 "J1" H 1100 3650 50  0000 L CNN
 F 1 "Power" H 1900 3650 50  0000 R CNN
-F 2 "Ratfink_Connectors_USB:USB_C_Receptacle_Amphenol_12401548E4-2A_CircularHoles" H 1650 2200 50  0001 C CNN
+F 2 "Connectors_USB:USB_C_Receptacle_Amphenol_12401548E4-2A_CircularHoles" H 1650 2200 50  0001 C CNN
 F 3 "" H 1650 2200 50  0001 C CNN
 	1    1500 2200
@@
 F 0 "J2" H 1100 7150 50  0000 L CNN
 F 1 "UFP" H 1900 7150 50  0000 R CNN
-F 2 "Ratfink_Connectors_USB:USB_C_Receptacle_Amphenol_12401548E4-2A_CircularHoles" H 1650 5700 50  0001 C CNN
+F 2 "Connectors_USB:USB_C_Receptacle_Amphenol_12401548E4-2A_CircularHoles" H 1650 5700 50  0001 C CNN
 F 3 "" H 1650 5700 50  0001 C CNN
 	1    1500 5700

Commit message: Use USB-C PCB edge receptacles
Since I've had problems in the past with fab houses not making the tiny
holes for USB Type-C receptacles properly, I started looking for a
solution that would ensure I can reliably make these boards.  Inspired
by https://hackaday.io/project/28516-business-card-gamepad, I created
USB Type-C receptacles for the PCB edge in KiCad.  Now I don't have to
populate the receptacles at all (forgoing the shield pads, which were
unreliable in my testing, and did not impact functionality), meaning the
Wye boards are easier and cheaper to make.  You know what that means:
price reduction!

This updates the project to recent KiCad 5 nightlies.
Parts:
- J1, J2: footprint Connectors_USB:USB_C_Receptacle_Amphenol_12401548E4-2A_CircularHoles -> Connector_USB_C_PCBEdge:USB_C_Receptacle_PCBEdge_Alt_ShieldPads; symbol USB_C_Receptacle -> Connector:USB_C_Receptacle
- MK1, MK2: symbol Mounting_Hole_PAD -> Mechanical:Mounting_Hole_PAD
- P1: symbol USB_C_Plug -> Connector:USB_C_Plug
- R1, R2: footprint Resistors_SMD:R_0805 -> Resistor_SMD:R_0805_2012Metric; symbol R -> Device:R
Changed lines of the file:
@@
-EESchema Schematic File Version 2
-LIBS:power
-LIBS:device
-LIBS:transistors
-LIBS:conn
-LIBS:linear
-LIBS:regul
-LIBS:74xx
-LIBS:cmos4000
-LIBS:adc-dac
-LIBS:memory
-LIBS:xilinx
-LIBS:microcontrollers
-LIBS:dsp
-LIBS:microchip
-LIBS:analog_switches
-LIBS:motorola
-LIBS:texas
-LIBS:intel
-LIBS:audio
-LIBS:interface
-LIBS:digital-audio
-LIBS:philips
-LIBS:display
-LIBS:cypress
-LIBS:siliconi
-LIBS:opto
-LIBS:atmel
-LIBS:contrib
-LIBS:valves
-LIBS:mechanical
+EESchema Schematic File Version 4
 LIBS:pd-buddy-wye-cache
-EELAYER 25 0
+EELAYER 26 0
 EELAYER END
 $Descr USLetter 11000 8500
@@
 Title "PD Buddy Wye"
 Date "2017-08-06"
-Rev "v1.1"
+Rev "v1.2"
 Comp ""
 Comment1 ""
@@
 $EndDescr
 $Comp
-L USB_C_Receptacle J1
+L Connector:USB_C_Receptacle J1
 U 1 1 59860B95
 P 1500 2200
 F 0 "J1" H 1100 3650 50  0000 L CNN
 F 1 "Power" H 1900 3650 50  0000 R CNN
-F 2 "Connectors_USB:USB_C_Receptacle_Amphenol_12401548E4-2A_CircularHoles" H 1650 2200 50  0001 C CNN
+F 2 "Connector_USB_C_PCBEdge:USB_C_Receptacle_PCBEdge_Alt_ShieldPads" H 1650 2200 50  0001 C CNN
 F 3 "" H 1650 2200 50  0001 C CNN
 	1    1500 2200
@@
 $EndComp
 $Comp
-L USB_C_Plug P1
+L Connector:USB_C_Plug P1
 U 1 1 59860CDD
 P 5700 4000
@@
 $EndComp
 $Comp
-L VBUS #PWR01
+L power:VBUS #PWR01
 U 1 1 59860D74
 P 2200 800
@@
 $EndComp
 $Comp
-L GND #PWR02
+L power:GND #PWR02
 U 1 1 59860ED6
 P 1600 4000
@@
 $EndComp
 $Comp
-L GND #PWR03
+L power:GND #PWR03
 U 1 1 59860F61
 P 1600 7500
@@
 $EndComp
 $Comp
-L GND #PWR04
+L power:GND #PWR04
 U 1 1 59860FEA
 P 5600 5800
@@
 $EndComp
 $Comp
-L VBUS #PWR05
+L power:VBUS #PWR05
 U 1 1 59861053
 P 5000 2600
@@
 	2200 1200 2100 1200
 Wire Wire Line
-	2200 800  2200 1200
+	2200 800  2200 900
 Wire Wire Line
 	2100 900  2200 900
@@
 Connection ~ 2200 1100
 Wire Wire Line
-	1600 3800 1600 4000
-Wire Wire Line
-	1200 3900 1600 3900
+	1600 3800 1600 3900
+Wire Wire Line
+	1200 3900 1300 3900
 Wire Wire Line
 	1200 3900 1200 3800
@@
 Connection ~ 1500 3900
 Wire Wire Line
-	1600 7300 1600 7500
-Wire Wire Line
-	1200 7400 1600 7400
+	1600 7300 1600 7400
+Wire Wire Line
+	1200 7400 1300 7400
 Wire Wire Line
 	1200 7400 1200 7300
@@
 Connection ~ 1500 7400
 Wire Wire Line
-	5600 5600 5600 5800
-Wire Wire Line
-	5600 5700 6000 5700
+	5600 5600 5600 5700
+Wire Wire Line
+	5600 5700 5700 5700
 Wire Wire Line
 	6000 5700 6000 5600
@@
 	5000 3000 5100 3000
 Wire Wire Line
-	5000 2600 5000 3000
+	5000 2600 5000 2700
 Wire Wire Line
 	5100 2700 5000 2700
@@
 	2200 5500 2200 5400
 Wire Wire Line
-	2100 5400 4800 5400
+	2100 5400 2200 5400
 Wire Wire Line
 	4800 5400 4800 3700
@@
 	2200 5200 2200 5300
 Wire Wire Line
-	2100 5300 4700 5300
+	2100 5300 2200 5300
 Wire Wire Line
 	4700 5300 4700 3500
@@
 	4700 1500 2100 1500
 $Comp
-L Mounting_Hole_PAD MK1
+L Mechanical:Mounting_Hole_PAD MK1
 U 1 1 59861CE1
 P 5650 1500
@@
 $EndComp
 $Comp
-L GND #PWR06
+L power:GND #PWR06
 U 1 1 59861D42
 P 5650 1600
@@
 $EndComp
 $Comp
-L Mounting_Hole_PAD MK2
+L Mechanical:Mounting_Hole_PAD MK2
 U 1 1 59861F93
 P 5650 6600
@@
 $EndComp
 $Comp
-L GND #PWR07
+L power:GND #PWR07
 U 1 1 59861F99
 P 5650 6700
@@
 CC2P
 $Comp
-L USB_C_Receptacle J2
+L Connector:USB_C_Receptacle J2
 U 1 1 59860C73
 P 1500 5700
 F 0 "J2" H 1100 7150 50  0000 L CNN
 F 1 "UFP" H 1900 7150 50  0000 R CNN
-F 2 "Connectors_USB:USB_C_Receptacle_Amphenol_12401548E4-2A_CircularHoles" H 1650 5700 50  0001 C CNN
+F 2 "Connector_USB_C_PCBEdge:USB_C_Receptacle_PCBEdge_Alt_ShieldPads" H 1650 5700 50  0001 C CNN
 F 3 "" H 1650 5700 50  0001 C CNN
 	1    1500 5700
@@
 $EndComp
 $Comp
-L R R2
+L Device:R R2
 U 1 1 59863CCA
 P 2650 5000
 F 0 "R2" V 2730 5000 50  0000 C CNN
 F 1 "5.1k" V 2650 5000 50  0000 C CNN
-F 2 "Resistors_SMD:R_0805" V 2580 5000 50  0001 C CNN
+F 2 "Resistor_SMD:R_0805_2012Metric" V 2580 5000 50  0001 C CNN
 F 3 "" H 2650 5000 50  0001 C CNN
 	1    2650 5000
@@
 $EndComp
 $Comp
-L R R1
+L Device:R R1
 U 1 1 59863DDF
 P 2650 4900
 F 0 "R1" V 2730 4900 50  0000 C CNN
 F 1 "5.1k" V 2650 4900 50  0000 C CNN
-F 2 "Resistors_SMD:R_0805" V 2580 4900 50  0001 C CNN
+F 2 "Resistor_SMD:R_0805_2012Metric" V 2580 4900 50  0001 C CNN
 F 3 "" H 2650 4900 50  0001 C CNN
 	1    2650 4900
@@
 	2100 5000 2500 5000
 Wire Wire Line
-	2800 5000 3000 5000
+	2800 5000 2900 5000
 Wire Wire Line
 	2900 4900 2800 4900
 Connection ~ 2900 5000
 $Comp
-L GND #PWR08
+L power:GND #PWR08
 U 1 1 59863FAB
 P 3000 5000
@@
 Text Label 2200 5000 0    60   ~ 0
 CC2D
+Wire Wire Line
+	2200 900  2200 1000
+Wire Wire Line
+	2200 1000 2200 1100
+Wire Wire Line
+	2200 1100 2200 1200
+Wire Wire Line
+	1600 3900 1600 4000
+Wire Wire Line
+	1300 3900 1400 3900
+Wire Wire Line
+	1400 3900 1500 3900
+Wire Wire Line
+	1500 3900 1600 3900
+Wire Wire Line
+	1600 7400 1600 7500
+Wire Wire Line
+	1300 7400 1400 7400
+Wire Wire Line
+	1400 7400 1500 7400
+Wire Wire Line
+	1500 7400 1600 7400
+Wire Wire Line
+	5600 5700 5600 5800
+Wire Wire Line
+	5900 5700 6000 5700
+Wire Wire Line
+	5800 5700 5900 5700
+Wire Wire Line
+	5700 5700 5800 5700
+Wire Wire Line
+	5000 2700 5000 2800
+Wire Wire Line
+	5000 2800 5000 2900
+Wire Wire Line
+	5000 2900 5000 3000
+Wire Wire Line
+	2200 5400 4800 5400
+Wire Wire Line
+	2200 5300 4700 5300
+Wire Wire Line
+	2900 5000 3000 5000
 $EndSCHEMATC
